File: Mini Project/MINIP.kicad_sch (KiCad schematic)
At the start: 8 parts

Commit message: fix miniproject files
Parts:
- R1, R2: value R -> 220
Other:
- moved on the sheet: D1, D2, I2C_LCD1, R1, R2
Changed lines of the file:
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@@
 	(wire
 		(pts
-			(xy 175.26 78.74) (xy 179.07 78.74)
-		)
-		(stroke
-			(width 0)
-			(type default)
-		)
-	)
-	(wire
-		(pts
-			(xy 124.46 64.77) (xy 124.46 67.31)
+			(xy 184.15 106.68) (xy 187.96 106.68)
+		)
+		(stroke
+			(width 0)
+			(type default)
+		)
+	)
+	(wire
+		(pts
+			(xy 107.95 54.61) (xy 107.95 57.15)
 		)
 		(stroke
@@
 	(wire
 		(pts
-			(xy 127 64.77) (xy 127 67.31)
+			(xy 110.49 54.61) (xy 110.49 57.15)
 		)
 		(stroke
@@
 	(wire
 		(pts
-			(xy 154.94 99.06) (xy 158.75 99.06)
+			(xy 165.1 82.55) (xy 168.91 82.55)
 		)
 		(stroke
@@
 	(wire
 		(pts
-			(xy 132.08 64.77) (xy 132.08 67.31)
+			(xy 115.57 54.61) (xy 115.57 57.15)
 		)
 		(stroke
@@
 	(wire
 		(pts
-			(xy 173.99 99.06) (xy 177.8 99.06)
-		)
-		(stroke
-			(width 0)
-			(type default)
-		)
-	)
-	(wire
-		(pts
-			(xy 156.21 78.74) (xy 160.02 78.74)
-		)
-		(stroke
-			(width 0)
-			(type default)
-		)
-	)
-	(wire
-		(pts
-			(xy 129.54 64.77) (xy 129.54 67.31)
+			(xy 184.15 82.55) (xy 187.96 82.55)
+		)
+		(stroke
+			(width 0)
+			(type default)
+		)
+	)
+	(wire
+		(pts
+			(xy 165.1 106.68) (xy 168.91 106.68)
+		)
+		(stroke
+			(width 0)
+			(type default)
+		)
+	)
+	(wire
+		(pts
+			(xy 113.03 54.61) (xy 113.03 57.15)
 		)
 		(stroke
@@
 	)
 	(label "SCL"
-		(at 124.46 67.31 270)
+		(at 107.95 57.15 270)
 		(fields_autoplaced yes)
 		(effects
@@
 	)
 	(label "GND"
-		(at 179.07 78.74 0)
+		(at 187.96 106.68 0)
 		(fields_autoplaced yes)
 		(effects
@@
 	)
 	(label "D3"
-		(at 154.94 99.06 0)
+		(at 165.1 82.55 0)
 		(fields_autoplaced yes)
 		(effects
@@
 	)
 	(label "GND"
-		(at 132.08 67.31 270)
+		(at 115.57 57.15 270)
 		(fields_autoplaced yes)
 		(effects
@@
 	)
 	(label "SDA"
-		(at 127 67.31 270)
+		(at 110.49 57.15 270)
 		(fields_autoplaced yes)
 		(effects
@@
 	)
 	(label "GND"
-		(at 177.8 99.06 0)
+		(at 187.96 82.55 0)
 		(fields_autoplaced yes)
 		(effects
@@
 	)
 	(label "5V"
-		(at 129.54 67.31 270)
+		(at 113.03 57.15 270)
 		(fields_autoplaced yes)
 		(effects
@@
 	)
 	(label "D4"
-		(at 156.21 78.74 0)
+		(at 165.1 106.68 0)
 		(fields_autoplaced yes)
 		(effects
@@
 		(dnp no)
 		(fields_autoplaced yes)
-		(property "Reference" "#PWR01"
+		(property "Reference" "#PWR02"
 			(at 96.52 110.49 0)
 			(effects
@@
 			(project ""
 				(path "/f497d447-3b22-454f-a20d-31c90dc48ae0"
-					(reference "#PWR01")
+					(reference "#PWR02")
 					(unit 1)
 				)
@@
 		(dnp no)
 		(fields_autoplaced yes)
-		(property "Reference" "#FLG01"
+		(property "Reference" "#FLG02"
 			(at 92.71 112.395 0)
 			(effects
@@
 					(size 1.27 1.27)
 				)
+				(hide yes)
 			)
 		)
@@
 			(project "MINIP"
 				(path "/f497d447-3b22-454f-a20d-31c90dc48ae0"
-					(reference "#FLG01")
+					(reference "#FLG02")
 					(unit 1)
 				)
@@
 		(dnp no)
 		(fields_autoplaced yes)
-		(property "Reference" "#PWR02"
+		(property "Reference" "#PWR01"
 			(at 86.36 107.95 0)
 			(effects
@@
 			(project ""
 				(path "/f497d447-3b22-454f-a20d-31c90dc48ae0"
-					(reference "#PWR02")
+					(reference "#PWR01")
 					(unit 1)
 				)
@@
 	(symbol
 		(lib_id "Device:LED")
-		(at 171.45 78.74 180)
+		(at 180.34 106.68 180)
 		(unit 1)
 		(exclude_from_sim no)
@@
 		(fields_autoplaced yes)
 		(property "Reference" "D2"
-			(at 173.0375 85.09 0)
+			(at 181.9275 113.03 0)
 			(effects
 				(font
@@
 		)
 		(property "Value" "LED"
-			(at 173.0375 82.55 0)
+			(at 181.9275 110.49 0)
 			(effects
 				(font
@@
 		)
 		(property "Footprint" ""
-			(at 171.45 78.74 0)
+			(at 180.34 106.68 0)
 			(effects
 				(font
@@
 		)
 		(property "Datasheet" "~"
-			(at 171.45 78.74 0)
+			(at 180.34 106.68 0)
 			(effects
 				(font
@@
 		)
 		(property "Description" "Light emitting diode"
-			(at 171.45 78.74 0)
+			(at 180.34 106.68 0)
 			(effects
 				(font
@@
 	(symbol
 		(lib_id "Device:R")
-		(at 162.56 99.06 270)
+		(at 172.72 82.55 270)
 		(unit 1)
 		(exclude_from_sim no)
@@
 		(fields_autoplaced yes)
 		(property "Reference" "R1"
-			(at 162.56 92.71 90)
-			(effects
-				(font
-					(size 1.27 1.27)
-				)
-			)
-		)
-		(property "Value" "R"
-			(at 162.56 95.25 90)
+			(at 172.72 76.2 90)
+			(effects
+				(font
+					(size 1.27 1.27)
+				)
+			)
+		)
+		(property "Value" "220"
+			(at 172.72 78.74 90)
 			(effects
 				(font
@@
 		)
 		(property "Footprint" ""
-			(at 162.56 97.282 90)
+			(at 172.72 80.772 90)
 			(effects
 				(font
@@
 		)
 		(property "Datasheet" "~"
-			(at 162.56 99.06 0)
+			(at 172.72 82.55 0)
 			(effects
 				(font
@@
 		)
 		(property "Description" "Resistor"
-			(at 162.56 99.06 0)
+			(at 172.72 82.55 0)
 			(effects
 				(font
@@
 	(symbol
 		(lib_id "minip:I2C_LCD")
-		(at 128.27 59.69 90)
+		(at 111.76 49.53 90)
 		(unit 1)
 		(exclude_from_sim no)
@@
 		(fields_autoplaced yes)
 		(property "Reference" "I2C_LCD1"
-			(at 134.62 57.7849 90)
+			(at 118.11 47.6249 90)
 			(effects
 				(font
@@
 		)
 		(property "Value" "~"
-			(at 134.62 59.69 90)
+			(at 118.11 49.53 90)
 			(effects
 				(font
@@
 		)
 		(property "Footprint" ""
-			(at 128.27 59.69 0)
+			(at 111.76 49.53 0)
 			(effects
 				(font
@@
 		)
 		(property "Datasheet" ""
-			(at 128.27 59.69 0)
+			(at 111.76 49.53 0)
 			(effects
 				(font
@@
 		)
 		(property "Description" ""
-			(at 128.27 59.69 0)
+			(at 111.76 49.53 0)
 			(effects
 				(font
@@
 		(dnp no)
 		(fields_autoplaced yes)
-		(property "Reference" "#FLG02"
+		(property "Reference" "#FLG01"
 			(at 92.71 106.045 0)
 			(effects
@@
 					(size 1.27 1.27)
 				)
+				(hide yes)
 			)
 		)
@@
 			(project "MINIP"
 				(path "/f497d447-3b22-454f-a20d-31c90dc48ae0"
-					(reference "#FLG02")
+					(reference "#FLG01")
 					(unit 1)
 				)
@@
 	(symbol
 		(lib_id "Device:LED")
-		(at 170.18 99.06 180)
+		(at 180.34 82.55 180)
 		(unit 1)
 		(exclude_from_sim no)
@@
 		(fields_autoplaced yes)
 		(property "Reference" "D1"
-			(at 171.7675 105.41 0)
+			(at 181.9275 88.9 0)
 			(effects
 				(font
@@
 		)
 		(property "Value" "LED"
-			(at 171.7675 102.87 0)
+			(at 181.9275 86.36 0)
 			(effects
 				(font
@@
 		)
 		(property "Footprint" ""
-			(at 170.18 99.06 0)
+			(at 180.34 82.55 0)
 			(effects
 				(font
@@
 		)
 		(property "Datasheet" "~"
-			(at 170.18 99.06 0)
+			(at 180.34 82.55 0)
 			(effects
 				(font
@@
 		)
 		(property "Description" "Light emitting diode"
-			(at 170.18 99.06 0)
+			(at 180.34 82.55 0)
 			(effects
 				(font
@@
 	(symbol
 		(lib_id "Device:R")
-		(at 163.83 78.74 270)
+		(at 172.72 106.68 270)
 		(unit 1)
 		(exclude_from_sim no)
@@
 		(fields_autoplaced yes)
 		(property "Reference" "R2"
-			(at 163.83 72.39 90)
-			(effects
-				(font
-					(size 1.27 1.27)
-				)
-			)
-		)
-		(property "Value" "R"
-			(at 163.83 74.93 90)
+			(at 172.72 100.33 90)
+			(effects
+				(font
+					(size 1.27 1.27)
+				)
+			)
+		)
+		(property "Value" "220"
+			(at 172.72 102.87 90)
 			(effects
 				(font
@@
 		)
 		(property "Footprint" ""
-			(at 163.83 76.962 90)
+			(at 172.72 104.902 90)
 			(effects
 				(font
@@
 		)
 		(property "Datasheet" "~"
-			(at 163.83 78.74 0)
+			(at 172.72 106.68 0)
 			(effects
 				(font
@@
 		)
 		(property "Description" "Resistor"
-			(at 163.83 78.74 0)
-			(effects
-				(font
+			(at 172.72 106.68 0)
+			(effects
+				(font
