File: Mini Project/backup/MINIP.kicad_pcb (KiCad board)
At the start: 2 copper layers, 58 x 61.5 mm, 9 parts

Commit message: a
Routing:
- net GND: track 1.72 -> 93.6 mm
Changed lines of the file:
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@@
+	)
+	(segment
+		(start 147.712 69.328)
+		(end 147.712 64.212)
+		(width 0.5)
+		(layer "F.Cu")
+		(net 3)
+	)
+	(segment
+		(start 145 72.04)
+		(end 147.712 69.328)
+		(width 0.5)
+		(layer "F.Cu")
+		(net 3)
+	)
+	(segment
+		(start 147.712 64.212)
+		(end 146.5 63)
+		(width 0.5)
+		(layer "F.Cu")
+		(net 3)
+	)
+	(segment
+		(start 145 72.04)
+		(end 145 86.6625)
+		(width 0.5)
+		(layer "B.Cu")
+		(net 3)
 	)
 	(segment
 		(start 144.96 98)
 		(end 144.53 98.43)
+		(width 0.5)
+		(layer "B.Cu")
+		(net 3)
+	)
+	(segment
+		(start 144.57 98.39)
+		(end 144.57 103.89)
+		(width 0.5)
+		(layer "B.Cu")
+		(net 3)
+	)
+	(segment
+		(start 149.028 60.472)
+		(end 146.5 63)
 		(width 0.5)
 		(layer "B.Cu")
@@
 	)
 	(segment
+		(start 154.5 60.472)
+		(end 149.028 60.472)
+		(width 0.5)
+		(layer "B.Cu")
+		(net 3)
+	)
+	(segment
+		(start 145 86.6625)
+		(end 146.555 88.2175)
+		(width 0.5)
+		(layer "B.Cu")
+		(net 3)
+	)
+	(segment
+		(start 191.672 60.472)
+		(end 154.5 60.472)
+		(width 0.5)
+		(layer "B.Cu")
+		(net 3)
+	)
+	(segment
+		(start 144.96 86.7025)
+		(end 144.96 97.5)
+		(width 0.5)
+		(layer "B.Cu")
+		(net 3)
+	)
+	(segment
 		(start 144.96 98)
 		(end 144.57 98.39)
 		(width 0.5)
 		(layer "B.Cu")
+		(net 3)
+	)
+	(segment
+		(start 193 61.8)
+		(end 191.672 60.472)
+		(width 0.5)
+		(layer "B.Cu")
